File: Hardware/PROIECT_TSC.brd (EAGLE design)
At the start: 175.7 x 120 mm, 103 parts, among them IC1 XC6220A331MR-G, IC2 BD5229G-TR, J1 FH34SRJ-24S-0.5SH_99_, J2 SAMACSYS_PARTS_USB4110-GF-A, J3 QWIIC_RIGHT_ANGLE, J4 112A-TAAR-R03_ATTEND, Q1 20V/4.2A/52mΩ/1.4W, Q2 20V/4.2A/52mΩ/1.4W, Q3 SI1308EDL-T1-GE3, U1 W25Q512JVEIQ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

Commit message: Add files via upload
Connections:
- net GND: now also R2.1
Routing:
- net EPD_3V3: track 78.3 -> 79.1 mm
- net GND: vias 12 -> 15
Changed lines of the file:
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@@
 <vertex x="0.0762" y="0.0762"/>
 </polygon>
+<via x="24.5" y="26.5" extent="1-16" drill="0.35" alwaysstop="yes">
+</via>
+<via x="60" y="36.5" extent="1-16" drill="0.35" alwaysstop="yes">
+</via>
+<via x="56" y="44.5" extent="1-16" drill="0.35" alwaysstop="yes">
+</via>
+<contactref element="R2" pad="1"/>
+<wire x1="58.928" y1="7.62" x2="63.5" y2="6.97" width="0" layer="19" extent="1-1"/>
 </signal>
 <signal name="VUSB">
@@
 <wire x1="22.75" y1="45.75" x2="22.75" y2="45.25" width="0.127" layer="1"/>
 <wire x1="150.25" y1="47" x2="150.42" y2="47.16" width="0.127" layer="1"/>
-<wire x1="22.75" y1="45.75" x2="22.5868" y2="45.86" width="0.127" layer="1"/>
+<wire x1="22.5868" y1="45.86" x2="22.75" y2="45.75" width="0.127" layer="1"/>
 </signal>
 <signal name="USB_D+">
@@
 <wire x1="24" y1="45.75" x2="24.25" y2="45.5" width="0.127" layer="1"/>
 <wire x1="150.25" y1="49.25" x2="150.42" y2="49.06" width="0.127" layer="1"/>
-<wire x1="24" y1="45.75" x2="23.8568" y2="45.86" width="0.127" layer="1"/>
+<wire x1="23.8568" y1="45.86" x2="24" y2="45.75" width="0.127" layer="1"/>
 <via x="104.75" y="53" extent="1-16" drill="0.3">
 </via>
@@
 <wire x1="46.25" y1="31" x2="43.25" y2="31" width="0.127" layer="1"/>
 <wire x1="43.25" y1="31" x2="43.25" y2="30.86" width="0.127" layer="1"/>
-<wire x1="46.25" y1="31" x2="46.33" y2="30.86" width="0.127" layer="1"/>
+<wire x1="46.33" y1="30.86" x2="46.25" y2="31" width="0.127" layer="1"/>
 <wire x1="46.5" y1="31" x2="48.25" y2="31" width="0.127" layer="1"/>
 <wire x1="48.25" y1="31" x2="48.41" y2="30.86" width="0.127" layer="1"/>
-<wire x1="46.5" y1="31" x2="46.33" y2="30.86" width="0.127" layer="1"/>
+<wire x1="46.33" y1="30.86" x2="46.5" y2="31" width="0.127" layer="1"/>
 <wire x1="71.75" y1="14.75" x2="70" y2="14.75" width="0.127" layer="1"/>
 <wire x1="70" y1="14.75" x2="69.89" y2="14.6" width="0.127" layer="1"/>
@@
 <wire x1="77.25" y1="45" x2="76" y2="43.75" width="0.127" layer="1"/>
 <wire x1="101.75" y1="45" x2="77.25" y2="45" width="0.127" layer="1"/>
-<wire x1="101.75" y1="45" x2="101.76" y2="45.07" width="0.127" layer="1"/>
+<wire x1="101.76" y1="45.07" x2="101.75" y2="45" width="0.127" layer="1"/>
 <wire x1="20.75" y1="109" x2="20.5" y2="108.75" width="0.127" layer="1"/>
 <wire x1="27.25" y1="109" x2="20.75" y2="109" width="0.127" layer="1"/>
@@
 <wire x1="72.5" y1="29.5" x2="74.75" y2="27.25" width="0.127" layer="1"/>
 <wire x1="48.5" y1="29.5" x2="72.5" y2="29.5" width="0.127" layer="1"/>
-<wire x1="48.5" y1="29.5" x2="48.41" y2="29.56" width="0.127" layer="1"/>
+<wire x1="48.41" y1="29.56" x2="48.5" y2="29.5" width="0.127" layer="1"/>
 <via x="81.75" y="15" extent="1-16" drill="0.3">
 </via>
@@
 <wire x1="83.75" y1="34.5" x2="88.25" y2="30" width="0.127" layer="1"/>
 <wire x1="48.25" y1="34.5" x2="83.75" y2="34.5" width="0.127" layer="1"/>
-<wire x1="48.25" y1="34.5" x2="48.12" y2="34.62" width="0.127" layer="1"/>
+<wire x1="48.12" y1="34.62" x2="48.25" y2="34.5" width="0.127" layer="1"/>
 <via x="82.25" y="15.5" extent="1-16" drill="0.3">
 </via>
@@
 <wire x1="78.5" y1="13.25" x2="78" y2="12.75" width="0.127" layer="16"/>
 <wire x1="78.5" y1="19" x2="78.5" y2="13.25" width="0.127" layer="16"/>
-<wire x1="82" y1="22.5" x2="78.5" y2="19" width="0.127" layer="16"/>
-<wire x1="82" y1="25.25" x2="82" y2="22.5" width="0.127" layer="16"/>
-<wire x1="84.5" y1="27.75" x2="82" y2="25.25" width="0.127" layer="16"/>
 <wire x1="84.5" y1="59.5" x2="84.5" y2="42.75" width="0.127" layer="16"/>
 <wire x1="84.5" y1="42.75" x2="84.5" y2="27.75" width="0.127" layer="16"/>
@@
 <via x="84.5" y="42.75" extent="1-16" drill="0.3">
 </via>
+<wire x1="81.5833" y1="22.0833" x2="78.5" y2="19" width="0.127" layer="16"/>
+<wire x1="84.5" y1="27.75" x2="81.5833" y2="24.8333" width="0.127" layer="16"/>
+<wire x1="81.5833" y1="24.8333" x2="81.5833" y2="22.0833" width="0.127" layer="16"/>
 </signal>
 <signal name="EPD_BUSY">
@@
 <wire x1="116.75" y1="2.5" x2="99.25" y2="20" width="0.127" layer="1"/>
 <wire x1="83.75" y1="14.25" x2="83.8" y2="14.15" width="0.127" layer="1"/>
-<wire x1="116.75" y1="2.5" x2="116.83" y2="2.2508" width="0.127" layer="1"/>
+<wire x1="116.83" y1="2.2508" x2="116.75" y2="2.5" width="0.127" layer="1"/>
 <wire x1="16.25" y1="65.5" x2="16.25" y2="63.5" width="0.127" layer="1"/>
 <wire x1="41" y1="65.5" x2="16.25" y2="65.5" width="0.127" layer="1"/>
@@
 <wire x1="34.75" y1="49.75" x2="38.25" y2="49.75" width="0.127" layer="1"/>
 <wire x1="102.75" y1="56" x2="102.83" y2="56.13" width="0.127" layer="1"/>
-<wire x1="34.75" y1="49.75" x2="34.74" y2="49.62" width="0.127" layer="1"/>
+<wire x1="34.74" y1="49.62" x2="34.75" y2="49.75" width="0.127" layer="1"/>
 <wire x1="21.5" y1="47.5" x2="21.5" y2="46" width="0.127" layer="1"/>
 <wire x1="33" y1="47.5" x2="21.5" y2="47.5" width="0.127" layer="1"/>
@@
 <wire x1="81.5" y1="15.75" x2="81.25" y2="15.75" width="0.127" layer="1"/>
 <wire x1="82.5" y1="16.75" x2="81.5" y2="15.75" width="0.127" layer="16"/>
-<wire x1="82.5" y1="23.25" x2="82.5" y2="20" width="0.127" layer="16"/>
+<wire x1="82" y1="23.25" x2="82" y2="20" width="0.127" layer="16"/>
 <wire x1="82.5" y1="20" x2="82.5" y2="19.75" width="0.127" layer="16"/>
 <wire x1="82.5" y1="19.75" x2="82.5" y2="16.75" width="0.127" layer="16"/>
-<wire x1="83.25" y1="24" x2="82.5" y2="23.25" width="0.127" layer="1"/>
+<wire x1="83.03301875" y1="24.28301875" x2="82" y2="23.25" width="0.127" layer="1"/>
 <wire x1="81.25" y1="14.25" x2="81.3" y2="14.15" width="0.127" layer="1"/>
-<wire x1="83.25" y1="24" x2="83.296" y2="23.94" width="0.127" layer="1"/>
+<wire x1="83.296" y1="23.94" x2="83.03301875" y2="24.28301875" width="0.127" layer="1"/>
 <wire x1="87" y1="17.75" x2="86.5" y2="18.25" width="0.127" layer="1"/>
 <wire x1="88" y1="17.75" x2="87" y2="17.75" width="0.127" layer="1"/>
@@
 <wire x1="78" y1="20" x2="77.75" y2="19.75" width="0.127" layer="1"/>
 <wire x1="81" y1="20" x2="78" y2="20" width="0.127" layer="1"/>
-<wire x1="82.5" y1="20" x2="81" y2="20" width="0.127" layer="16"/>
+<wire x1="82.5" y1="20" x2="82" y2="20" width="0.127" layer="16"/>
+<wire x1="82" y1="20" x2="81" y2="20" width="0.127" layer="16"/>
 <wire x1="75.25" y1="19.75" x2="75.2" y2="19.64" width="0.127" layer="1"/>
 <via x="81.5" y="15.75" extent="1-16" drill="0.3">
 </via>
-<via x="82.5" y="23.25" extent="1-16" drill="0.3">
+<via x="82" y="23.25" extent="1-16" drill="0.3">
 </via>
 <via x="85.25" y="19.5" extent="1-16" drill="0.3">
@@
 <wire x1="73.25" y1="20" x2="73" y2="20.25" width="0.127" layer="1"/>
 <wire x1="117.25" y1="57.5" x2="117.36" y2="57.64" width="0.127" layer="1"/>
-<wire x1="73.25" y1="20" x2="73.34" y2="19.9" width="0.127" layer="1"/>
+<wire x1="73.34" y1="19.9" x2="73.25" y2="20" width="0.127" layer="1"/>
 <via x="114.5" y="55.25" extent="1-16" drill="0.3">
 </via>
