File: Hardware/PROIECT_TSC.sch (EAGLE design)
At the start: 103 parts, among them IC1 XC6220A331MR-G, IC2 BD5229G-TR, J1 FH34SRJ-24S-0.5SH_99_, J2 SAMACSYS_PARTS_USB4110-GF-A, J3 QWIIC_RIGHT_ANGLE, J4 112A-TAAR-R03_ATTEND, Q1 20V/4.2A/52mΩ/1.4W, Q2 20V/4.2A/52mΩ/1.4W, Q3 SI1308EDL-T1-GE3, U1 W25Q512JVEIQ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

Commit message: Add files via upload
Connections:
- net GND: now also R2.1
Other:
- moved on the sheet: EPD_C11
Changed lines of the file:
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@@
 <attribute name="VALUE" x="121.539" y="128.524" size="1.016" layer="96" rot="R180"/>
 </instance>
-<instance part="EPD_C11" gate="G$1" x="104.14" y="132.08" smashed="yes" rot="R90">
-<attribute name="NAME" x="113.919" y="133.604" size="1.016" layer="95" rot="R180"/>
-<attribute name="VALUE" x="103.759" y="131.064" size="1.016" layer="96" rot="R180"/>
+<instance part="EPD_C11" gate="G$1" x="101.6" y="132.08" smashed="yes" rot="R90">
+<attribute name="NAME" x="111.379" y="133.604" size="1.016" layer="95" rot="R180"/>
+<attribute name="VALUE" x="101.219" y="131.064" size="1.016" layer="96" rot="R180"/>
 </instance>
 <instance part="EPD_C12" gate="G$1" x="96.52" y="134.62" smashed="yes" rot="R90">
@@
 <pinref part="SUPPLY15" gate="G$1" pin="GND"/>
 <wire x1="86.36" y1="162.56" x2="86.36" y2="167.64" width="0.1524" layer="91"/>
-<wire x1="86.36" y1="167.64" x2="93.98" y2="167.64" width="0.1524" layer="91"/>
+<wire x1="86.36" y1="167.64" x2="96.52" y2="167.64" width="0.1524" layer="91"/>
+<pinref part="R2" gate="G$1" pin="1"/>
 </segment>
 <segment>
@@
 <pinref part="EPD_C12" gate="G$1" pin="1"/>
 <pinref part="EPD_C11" gate="G$1" pin="1"/>
-<wire x1="101.6" y1="132.08" x2="91.44" y2="132.08" width="0.1524" layer="91"/>
+<wire x1="99.06" y1="132.08" x2="91.44" y2="132.08" width="0.1524" layer="91"/>
 <wire x1="91.44" y1="134.62" x2="91.44" y2="132.08" width="0.1524" layer="91"/>
 <wire x1="91.44" y1="132.08" x2="91.44" y2="129.54" width="0.1524" layer="91"/>
 <wire x1="91.44" y1="129.54" x2="111.76" y2="129.54" width="0.1524" layer="91"/>
 <pinref part="EPD_C10" gate="G$1" pin="1"/>
-<junction x="91.44" y="134.62"/>
-<junction x="91.44" y="132.08"/>
 <pinref part="EPD_C5" gate="G$1" pin="1"/>
 <wire x1="93.98" y1="111.76" x2="91.44" y2="111.76" width="0.1524" layer="91"/>
 <wire x1="91.44" y1="111.76" x2="91.44" y2="119.38" width="0.1524" layer="91"/>
-<junction x="91.44" y="129.54"/>
 <pinref part="EPD_C6" gate="G$1" pin="1"/>
 <wire x1="91.44" y1="119.38" x2="91.44" y2="121.92" width="0.1524" layer="91"/>
@@
 <wire x1="91.44" y1="127" x2="91.44" y2="129.54" width="0.1524" layer="91"/>
 <wire x1="111.76" y1="119.38" x2="91.44" y2="119.38" width="0.1524" layer="91"/>
-<junction x="91.44" y="119.38"/>
 <pinref part="EPD_C7" gate="G$1" pin="1"/>
 <wire x1="99.06" y1="121.92" x2="91.44" y2="121.92" width="0.1524" layer="91"/>
-<junction x="91.44" y="121.92"/>
 <pinref part="EPD_C8" gate="G$1" pin="1"/>
 <wire x1="111.76" y1="124.46" x2="91.44" y2="124.46" width="0.1524" layer="91"/>
-<junction x="91.44" y="124.46"/>
 <pinref part="EPD_C9" gate="G$1" pin="1"/>
 <wire x1="99.06" y1="127" x2="91.44" y2="127" width="0.1524" layer="91"/>
+<junction x="91.44" y="134.62"/>
+<junction x="91.44" y="132.08"/>
+<junction x="91.44" y="129.54"/>
+<junction x="91.44" y="119.38"/>
+<junction x="91.44" y="121.92"/>
+<junction x="91.44" y="124.46"/>
 <junction x="91.44" y="127"/>
 </segment>
@@
 <wire x1="127" y1="132.08" x2="121.92" y2="132.08" width="0.1524" layer="91"/>
 <pinref part="EPD_C11" gate="G$1" pin="2"/>
-<wire x1="121.92" y1="132.08" x2="109.22" y2="132.08" width="0.1524" layer="91"/>
+<wire x1="121.92" y1="132.08" x2="106.68" y2="132.08" width="0.1524" layer="91"/>
 <wire x1="121.92" y1="132.08" x2="121.92" y2="137.16" width="0.1524" layer="91"/>
 <label x="121.92" y="137.16" size="1.016" layer="95" rot="R90" xref="yes"/>
